File: esp_i2c.kicad_pcb (KiCad board)
At the start: 2 copper layers, 50 x 30 mm, 19 parts, among them J1 FTDI, J2 Screw_Terminal_01x02, J3 USB_B_Micro, J4 Conn_02x08_Counter_Clockwise, SW1 BOOTSEL, U1 ESP32-WROOM-32, U2 TLV1117-33

Commit message: v0.2
Parts:
- removed TP1, TP2: TestPoint, TestPoint:TestPoint_Pad_D1.0mm
- added D1: D, Diode_SMD:D_SOD-323, F.Cu at (119.5, 84.0)
- added D2: D, Diode_SMD:D_SOD-323, F.Cu at (96.9, 83.4)
- added J5: Conn_01x02_Male, Connector_PinHeader_2.54mm:PinHeader_1x02_P2.54mm_Vertical, F.Cu at (92.0, 87.9)
- added SW2: RST, Button_Switch_THT:SW_PUSH_6mm_H5mm, F.Cu at (93.6, 68.3)
- H1, H2, H3, H4: footprint MountingHole:MountingHole_3.5mm_Pad -> MountingHole:MountingHole_3.2mm_M3_ISO7380_Pad
- J1: footprint Connector_PinHeader_2.54mm:PinHeader_1x05_P2.54mm_Vertical -> Connector_PinHeader_2.54mm:PinHeader_1x06_P2.54mm_Vertical
- J3: value USB_B_Micro -> Molex 105017-0001
- R1: value 10k -> 1k
- SW1: value BOOTSEL -> DL
- U2: value TLV1117-33 -> TLV1117LV33
- moved C3 9.29 mm to (83.7, 68.7), turned to 270 degrees
- moved C5 7.80 mm to (85.7, 81.2), turned to 0 degrees
- moved C2 7.58 mm to (92.3, 62.1)
- moved R1 5.91 mm to (85.8, 68.7)
- moved C1 3.78 mm to (89.6, 62.1)
- moved SW1 1.40 mm to (86.1, 72.1)
- moved J1 1.10 mm to (123.6, 81.2)
- moved H3 0.44 mm to (83.5, 63.5)
- moved H1 0.44 mm to (126.5, 63.5)
- moved H4 0.43 mm to (83.5, 86.5)
- moved H2 0.43 mm to (126.5, 86.5)
- moved C4 0.10 mm to (96.9, 81.4)
Connections:
- C3 pad 2: Net-(C3-Pad2) -> RST
- C4 pad 2: VBUS -> Net-(C4-Pad2)
- J1 pad 3: (no net) -> Net-(D1-Pad2)
- J3 pad 1: VBUS -> Net-(D2-Pad2)
- J4 pad 3: MOSI -> SS
- J4 pad 5: MISO -> SCLK
- J4 pad 7: SCLK -> MISO
- J4 pad 9: SS -> MOSI
- R1 pad 2: Net-(C3-Pad2) -> RST
- U1 pad 12: (no net) -> GPIO2
- U1 pad 13: (no net) -> GPIO3
- U1 pad 14: (no net) -> GPIO4
- U1 pad 17: U1_RX -> (no net)
- U1 pad 18: U1_TX -> (no net)
- U1 pad 19: SS -> (no net)
- U1 pad 20: SCLK -> (no net)
- U1 pad 21: MISO -> (no net)
- U1 pad 22: MOSI -> (no net)
- U1 pad 27: GPIO4 -> U1_RX
- U1 pad 28: GPIO3 -> U1_TX
- U1 pad 29: GPIO2 -> SS
- U1 pad 3: Net-(C3-Pad2) -> RST
- U1 pad 30: GPIO1 -> SCLK
- U1 pad 31: GPIO0 -> MISO
- U1 pad 37: (no net) -> MOSI
- U1 pad 8: (no net) -> GPIO0
- U1 pad 9: (no net) -> GPIO1
- U2 pad 3: VBUS -> Net-(C4-Pad2)
- U2 pad 4: (no net) -> VDD
Routing:
- net RST: track 0.00 -> 55.8 mm
- net GPIO3: track 4.23 -> 22.3 mm, vias 0 -> 1
- net GPIO4: track 3.71 -> 21.8 mm, vias 0 -> 1
- net GPIO2: track 5.18 -> 22.8 mm, vias 0 -> 1
- net GPIO1: track 6.16 -> 22.7 mm, vias 0 -> 1
- net GPIO0: track 7.43 -> 23.9 mm, vias 0 -> 1
- net SS: track 21.3 -> 8.90 mm, vias 1 -> 0
- net U1_TX: track 23.7 -> 11.7 mm
- net SCLK: track 19.0 -> 7.46 mm, vias 1 -> 0
- net Net-(C3-Pad2): track 11.2 -> 0.00 mm
- net Net-(C4-Pad2): track 0.00 -> 9.97 mm
- net MISO: track 16.7 -> 6.93 mm, vias 1 -> 0
- net RX: track 18.1 -> 27.6 mm, vias 0 -> 1
- net Net-(D1-Pad2): track 0.00 -> 9.14 mm
- net GND: track 41.0 -> 49.0 mm, vias 22 -> 18
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- added copper zone on B.Cu, net VDD
Other:
- board text added: "esp32_sens v0.2"
- board text removed: "esp32_sens v0.1"
