File: esp_i2c.sch (KiCad schematic (older format))
At the start: 19 parts, among them J1 FTDI, J2 Screw_Terminal_01x02, J3 USB_B_Micro, J4 Conn_02x08_Counter_Clockwise, SW1 BOOTSEL, U1 ESP32-WROOM-32, U2 TLV1117-33

Commit message: Update esp_i2c.sch
Parts:
- J3: value USB_B_Micro -> Molex 105017-0001
- U2: value TLV1117-33 -> TLV1117LV33
Changed lines of the file:
@@
 P 5000 1350
 F 0 "U2" H 5000 1592 50  0000 C CNN
-F 1 "TLV1117-33" H 5000 1501 50  0000 C CNN
+F 1 "TLV1117LV33" H 5000 1501 50  0000 C CNN
 F 2 "Package_TO_SOT_SMD:SOT-223" H 5000 1350 50  0001 C CNN
 F 3 "http://www.ti.com/lit/ds/symlink/tlv1117.pdf" H 5000 1350 50  0001 C CNN
@@
 P 6500 1250
 F 0 "J3" H 6557 1717 50  0000 C CNN
-F 1 "USB_B_Micro" H 6557 1626 50  0000 C CNN
+F 1 "Molex 105017-0001" H 6557 1626 50  0000 C CNN
 F 2 "Connector_USB:USB_Micro-B_Molex-105017-0001" H 6650 1200 50  0001 C CNN
 F 3 "~" H 6650 1200 50  0001 C CNN

Commit message: v0.2
Parts:
- removed TP1, TP2: TestPoint, TestPoint:TestPoint_Pad_D1.0mm, symbol Connector:TestPoint
- added D1, D2: D, Diode_SMD:D_SOD-323, symbol Device:D
- added J5: Conn_01x02_Male, Connector_PinHeader_2.54mm:PinHeader_1x02_P2.54mm_Vertical, symbol Connector:Conn_01x02_Male
- added SW2: RST, Button_Switch_THT:SW_PUSH_6mm_H5mm, symbol Switch:SW_Push
- H1, H2, H3, H4: footprint MountingHole:MountingHole_3.5mm_Pad -> MountingHole:MountingHole_3.2mm_M3_ISO7380_Pad
- J1: footprint Connector_PinHeader_2.54mm:PinHeader_1x05_P2.54mm_Vertical -> Connector_PinHeader_2.54mm:PinHeader_1x06_P2.54mm_Vertical; symbol Connector:Conn_01x05_Male -> Connector:Conn_01x06_Male
- J2: footprint TerminalBlock_Phoenix:TerminalBlock_Phoenix_MPT-0,5-2-2.54_1x02_P2.54mm_Horizontal -> TerminalBlock_Phoenix:TerminalBlock_Phoenix_PT-1,5-2-5.0-H_1x02_P5.00mm_Horizontal
- R1: value 10k -> 1k
- SW1: value BOOTSEL -> DL
Connections:
- net labels added: RST
- wire segments 24 -> 30
- no-connect marks 8 -> 13
Other:
- moved on the sheet: C3, R1
